File: wurtelvin/fin_lights.kicad_sch (KiCad schematic)
At the start: 9 parts, among them J10 FIN_TOP, J8 FIN_REAR, J9 FIN_FRONT

Commit message: furhter pcb layout
Parts:
- added R16, R17, R18: 300, Resistor_SMD:R_0603_1608Metric, symbol Device:R
- renumbered C22 to C20, C20 to C21, C23 to C22, C21 to C23
Connections:
- net FF_DATA: now also R17.1; no longer J9.2 (Pin_2)
- net FR_DATA: now also R16.1; no longer J8.2 (Pin_2)
- net FT_DATA: now also R18.1; no longer J10.2 (Pin_2)
- new net: J8.2 (Pin_2), R16.2
- new net: J10.2 (Pin_2), R18.2
- new net: J9.2 (Pin_2), R17.2
