File: wurtelvin/power.kicad_sch (KiCad schematic)
At the start: 12 parts, among them U10 XL1509-5.0, U9 XL1509-3.3

Commit message: furhter pcb layout
Parts:
- removed D8, D9: 1N5820, Diode_THT:D_DO-201AD_P15.24mm_Horizontal, symbol Diode:1N5820
- added D8, D9: SS32, Diode_SMD:D_SMA, symbol Diode:SS32
- renumbered C27 to C26, C29 to C27, C26 to C28, C28 to C29
Connections:
- net GND: now also D8.2 (A), D9.2 (A)
- net at L8.1, U9.2 (OUT): now also D8.1 (K)
- net at L9.1, U10.2 (OUT): now also D9.1 (K)
