File: wurtelvin/wurtelvin.kicad_pcb (KiCad board)
At the start: 2 copper layers, 40 x 130 mm, 93 parts, among them J1 BATT, J10 FIN_TOP, J2 FRONT, J3 MIRRORS, J4 REAR TURNERS, J5 REAR, J6 BTN_BRK, J7 btn_handle, J8 FIN_REAR, J9 FIN_FRONT, SW1 ON/OFF, SW2 DAYLIGHT, SW3 DIM, SW4 REAR, U1 STM32F103C8Tx, U10 XL1509-5.0, U2 AL8860WT, U3 AL8860WT, U4 AL8860WT, U5 AL8860WT, U6 AL8860WT, U7 AL8860WT, U8 AL8860WT, U9 XL1509-3.3, Y1 8MHz

Commit message: started pcb layout for connector and 3v3 and 5v step-down
Parts:
- removed SW3: DIM, Library:KNX1
- J7: value btn_handle -> BTN_HANDLE
- SW1: value ON/OFF -> SW_DPDT_x2; footprint Library:KNX1 -> Library:ANT_2x3
- SW2, SW4: footprint Library:KNX1 -> Library:ANT_1x3
- moved J6 131.0 mm to (137.4, 147.9)
- moved J5 120.3 mm to (121.9, 139.7), turned to -90 degrees
- moved J4 117.4 mm to (122.1, 125.1), turned to -90 degrees
- moved J7 90.0 mm to (121.8, 107.1), turned to -90 degrees
- moved J1 89.6 mm to (121.8, 80.3), turned to -90 degrees
- moved J10 88.1 mm to (148.3, 90.8), turned to 90 degrees
- moved J9 87.3 mm to (148.3, 77.8), turned to 90 degrees
- moved J8 86.2 mm to (148.3, 63.9), turned to 90 degrees
- moved SW1 81.4 mm to (123.0, 91.0)
- moved BZ1 80.0 mm to (126.9, 59.6), turned to 90 degrees
- moved J3 73.2 mm to (134.8, 31.0), turned to 180 degrees
- moved U9 69.4 mm to (133.0, 106.4), turned to 180 degrees
- moved D9 69.0 mm to (133.0, 129.0), turned to 90 degrees
- moved R1 67.8 mm to (121.3, 63.1), turned to 180 degrees
- moved C1 66.6 mm to (118.2, 63.1)
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Connections:
- SW1 pad 3: unconnected-(SW1-C-Pad3) -> +BATT
Routing:
- net +BATT: track 8.25 -> 35.1 mm
- net Net-(D8-K): track 0.00 -> 14.2 mm
- net Net-(D9-K): track 0.00 -> 13.8 mm
- net +5V: track 0.00 -> 11.0 mm
- net +3V3: track 0.00 -> 10.6 mm
- net Net-(J1-Pin_2): track 0.00 -> 7.97 mm
- net /BTN_DL: track 0.00 -> 6.68 mm

Commit message: furhter pcb layout
Parts:
- removed D8, D9: 1N5820, Diode_THT:D_DO-201AD_P15.24mm_Horizontal
- added D10: SS32, Diode_SMD:D_SMA, F.Cu at (135.6, 83.8)
- added D11: SS32, Diode_SMD:D_SMA, F.Cu at (131.7, 109.2)
- added R16: 300, Resistor_SMD:R_0603_1608Metric, F.Cu at (143.0, 82.9)
- added R17: 300, Resistor_SMD:R_0603_1608Metric, F.Cu at (142.0, 67.1)
- added R18: 300, Resistor_SMD:R_0603_1608Metric, F.Cu at (141.5, 93.8)
- C12, C13, C14, C15, C18, C5, C6, C7, C8, D1, D2, D3, D4, D7, L1, L2, L3, L4, L7, R10, R11, R12, R15, R5, R9, U1, U2, U3, U4, U5, U8, Y1: moved to B.Cu
- J7: value BTN_HANDLE -> btn_handle
- moved C15 120.9 mm to (130.8, 137.9), turned to 180 degrees
- moved U5 120.8 mm to (134.2, 136.7), turned to -90 degrees
- moved D4 119.2 mm to (126.6, 136.2), turned to 90 degrees
- moved R12 116.3 mm to (134.3, 139.8)
- moved C21 114.7 mm to (142.2, 70.2)
- moved L4 109.7 mm to (132.6, 130.9)
- moved D7 108.5 mm to (130.8, 152.2), turned to 180 degrees
- moved U8 108.1 mm to (134.7, 148.0)
- moved C18 106.5 mm to (137.2, 151.0)
- moved C19 104.3 mm to (141.1, 61.6), turned to -90 degrees
- moved C22 103.9 mm to (142.2, 73.7)
- moved L7 103.2 mm to (124.3, 143.7)
- moved C20 102.5 mm to (139.1, 66.1)
- moved U7 101.9 mm to (138.6, 138.3), turned to 90 degrees
- moved R15 100.7 mm to (138.1, 148.1), turned to 90 degrees
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Connections:
- net /front_lights/CTRL_DL renamed /CTRL_DL
- net /front_lights/CTRL_FH renamed /CTRL_FH
- net /front_lights/CTRL_FL renamed /CTRL_FL
- net /rear_lights/CTRL_BRK renamed /CTRL_BRK
- net /rear_lights/CTRL_REAR renamed /CTRL_REAR
- net /turning_lights/CTRL_TLL renamed /CTRL_TLL
- net /turning_lights/CTRL_TLR renamed /CTRL_TLR
- J10 pad 2: /fin_lights/FT_DATA -> Net-(J10-Pin_2)
- J8 pad 2: /fin_lights/FR_DATA -> Net-(J8-Pin_2)
- J9 pad 2: /fin_lights/FF_DATA -> Net-(J9-Pin_2)
- L1 pad 1: /front_lights/DL- -> /DL-
- L2 pad 1: /front_lights/FH- -> /FH-
- L3 pad 1: /front_lights/FL- -> /FL-
- L4 pad 1: /turning_lights/TLR- -> /TLR-
- L5 pad 1: /turning_lights/TLL- -> /TLL-
- L6 pad 1: /rear_lights/REAR- -> /REAR-
- L7 pad 1: /rear_lights/BRK- -> /BRK-
- R10 pad 2: /front_lights/FH+ -> /FH+
- R11 pad 2: /front_lights/FL+ -> /FL+
- R12 pad 2: /turning_lights/TLR+ -> /TLR+
- R13 pad 2: /turning_lights/TLL+ -> /TLL+
- R14 pad 2: /rear_lights/REAR+ -> /REAR+
- R15 pad 2: /rear_lights/BRK+ -> /BRK+
- R9 pad 2: /front_lights/DL+ -> /DL+
- U2 pad 4: /front_lights/DL+ -> /DL+
- U3 pad 4: /front_lights/FH+ -> /FH+
- U4 pad 4: /front_lights/FL+ -> /FL+
- U5 pad 4: /turning_lights/TLR+ -> /TLR+
- U6 pad 4: /turning_lights/TLL+ -> /TLL+
- U7 pad 4: /rear_lights/REAR+ -> /REAR+
- U8 pad 4: /rear_lights/BRK+ -> /BRK+
Routing:
- net +BATT: track 35.1 -> 104.5 mm
- net +5V: track 11.0 -> 52.8 mm
- net /REAR+: track 0.00 -> 31.0 mm
- net +3V3: track 10.6 -> 41.1 mm, vias 0 -> 1
- net /OSC_OUT: track 0.00 -> 17.0 mm
- net /OSC_IN: track 0.00 -> 16.8 mm
- net /BRK+: track 0.00 -> 16.5 mm, vias 0 -> 1
- net Net-(D7-A): track 0.00 -> 13.9 mm
- net /FH+: track 0.00 -> 13.0 mm
- net Net-(D6-A): track 0.00 -> 12.7 mm
- net Net-(D4-A): track 0.00 -> 11.7 mm
- net /FL+: track 0.00 -> 8.99 mm, vias 0 -> 1
- net /FL-: track 0.00 -> 8.36 mm
- net /BRK-: track 0.00 -> 8.10 mm, vias 0 -> 1
- net /TLR-: track 0.00 -> 7.50 mm, vias 0 -> 1
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- added copper zone on B.Cu, net GND
- added copper zone on F.Cu, net GND

Commit message: more routing
Parts:
- C10: renamed from C4; moved to B.Cu
- C16, C17, C25, D5, D6, L5, L6, L8, R13, R14, U6, U7, U9: moved to B.Cu
- C26: renamed from C27; moved to B.Cu
- C27: renamed from C29; moved to B.Cu
- C5: renamed from C9; moved to B.Cu
- C6: renamed from C2; moved to B.Cu
- C7: renamed from C10; moved to B.Cu
- C8: renamed from C3; moved to B.Cu
- C9: renamed from C11; moved to B.Cu
- D8: renamed from D11; moved to B.Cu
- R2: renamed from R7; moved to B.Cu
- R3: renamed from R8; moved to B.Cu
- R4: renamed from R2; moved to B.Cu
- R5: renamed from R6; moved to B.Cu
- R6: renamed from R3; moved to B.Cu
- R7: renamed from R4; moved to B.Cu
- moved C24 121.1 mm to (141.2, 86.6), turned to 90 degrees
- moved C22 110.3 mm to (148.6, 70.9), turned to 180 degrees
- moved D5 92.7 mm to (145.8, 79.4), turned to 180 degrees
- moved U6 91.8 mm to (149.2, 73.9)
- moved L5 89.2 mm to (142.2, 72.5)
- moved R13 83.9 mm to (152.8, 73.8), turned to 90 degrees
- moved C16 83.9 mm to (152.1, 76.6)
- moved R5 81.4 mm to (128.5, 111.2), turned to 180 degrees
- moved C9 81.3 mm to (128.5, 113.3)
- moved R4 80.3 mm to (118.3, 99.0), turned to 90 degrees
- moved R3 75.7 mm to (131.0, 102.4), turned to 180 degrees
- moved R6 75.3 mm to (118.2, 52.0), turned to 90 degrees
- moved C6 74.7 mm to (121.2, 98.2), turned to 180 degrees
- moved R7 71.0 mm to (126.5, 40.1)
- moved C8 70.4 mm to (119.2, 49.5), turned to 180 degrees
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- renumbered C5 to C1, C1 to C11, C6 to C2, C22 to C20, C20 to C21, C23 to C22, C21 to C23, C26 to C28, C28 to C29, C7 to C3, C8 to C4, D10 to D9, J2 to J1, J3 to J2, J4 to J3, J5 to J4, J6 to J5, J1 to J6, R5 to R1, R17 to R16, R16 to R17, R1 to R8, SW4 to SW2, SW2 to SW3
Connections:
- U1 pad 3: /OSC32_IN -> unconnected-(U1-PC14-Pad3)
- U1 pad 4: /OSC32_OUT -> unconnected-(U1-PC15-Pad4)
Routing:
- net +BATT: track 104.5 -> 237.9 mm, vias 0 -> 3
- net Net-(J2-Pin_3): track 0.00 -> 129.2 mm
- net +3V3: track 41.1 -> 155.8 mm
- net Net-(J2-Pin_7): track 0.00 -> 114.0 mm, vias 0 -> 2
- net /TLL-: track 0.00 -> 61.5 mm, vias 0 -> 1
- net /FF_DATA: track 0.00 -> 47.8 mm, vias 0 -> 1
- net /REAR+: track 31.0 -> 60.9 mm, vias 0 -> 1
- net Net-(J1-Pin_5): track 0.00 -> 27.1 mm
- net /FT_DATA: track 0.00 -> 26.0 mm, vias 0 -> 1
- net Net-(D3-A): track 3.42 -> 22.3 mm
- net /BTN_TLR: track 0.00 -> 18.8 mm, vias 0 -> 1
- net /REAR-: track 5.29 -> 20.2 mm, vias 0 -> 3
- net Net-(D5-A): track 0.00 -> 11.1 mm
- net Net-(J2-Pin_2): track 0.00 -> 10.3 mm
- net +5V: track 52.8 -> 61.9 mm
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
Commit message: finished routing except for control signals, switched to 4-layer pcb
Parts:
- moved C7 19.0 mm to (120.5, 109.2), turned to 0 degrees
- moved R2 17.6 mm to (120.5, 107.5)
- moved C28 11.8 mm to (129.8, 65.5)
- moved C29 11.0 mm to (129.8, 63.8)
- moved C5 10.0 mm to (121.0, 104.1)
- moved R3 10.0 mm to (121.0, 102.4)
- moved C10 4.05 mm to (126.5, 38.2), turned to 0 degrees
- moved D9 1.44 mm to (136.2, 82.5)
- moved C18 0.95 mm to (136.2, 151.0)
- moved D7 0.70 mm to (130.8, 151.5)
- moved C27 0.35 mm to (149.7, 103.0)
- moved U9 0.35 mm to (149.8, 107.8)
- moved C25 0.12 mm to (146.5, 111.5)
- moved C26 0.12 mm to (146.5, 113.2)
Routing:
- net /TLR+: track 0.00 -> 115.5 mm, vias 0 -> 1
- net /FR_DATA: track 0.00 -> 86.6 mm, vias 0 -> 3
- net +BATT: track 237.9 -> 308.4 mm, vias 3 -> 12
- net /HORN+: track 0.00 -> 68.6 mm, vias 0 -> 1
- net GND: track 0.00 -> 31.1 mm, vias 0 -> 434
- net +3V3: track 155.8 -> 186.0 mm, vias 1 -> 16
- net /TLL+: track 2.46 -> 29.9 mm, vias 0 -> 1
- net Net-(J1-Pin_3): track 0.00 -> 23.7 mm, vias 0 -> 2
- net /BTN_TLR: track 18.8 -> 8.08 mm
- net Net-(D2-A): track 3.92 -> 9.53 mm
- net /FF_DATA: track 47.8 -> 52.1 mm
- net /TLL-: track 61.5 -> 65.1 mm
- net /BRK+: track 16.5 -> 18.9 mm
- net /FH-: track 7.14 -> 9.17 mm
- net /FL-: track 8.36 -> 6.70 mm
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- added copper zone on In1.Cu, net GND
- added copper zone on In2.Cu, net GND
Other:
- copper layers 2 -> 4
